File: next-keyboard.kicad_pcb (KiCad board)
At the start: 2 copper layers, 95.2 x 92.9 mm, 37 parts, among them J1 MJ-4PP-9, J2 MJ-4PP-9, SW1 SW_PUSH, SW10 SW_PUSH, SW11 SW_PUSH, SW12 SW_PUSH, SW13 SW_PUSH, SW14 SW_PUSH, SW15 SW_PUSH, SW16 SW_PUSH, SW17 SW_PUSH, SW18 SW_PUSH, SW19 SW_PUSH, SW2 SW_PUSH, SW20 SW_PUSH, SW21 SW_SPDT, SW22 SW_SPDT, SW3 SW_PUSH, SW4 SW_PUSH, SW5 SW_PUSH, SW6 SW_PUSH, SW7 SW_PUSH, SW8 SW_PUSH, SW9 SW_PUSH, U1 MCP23017_SP, U2 MCP23017_SP

Commit message: produce
Parts:
- removed REF** (x4): MountingHole_3.2mm_M3, MountingHole:MountingHole_3.2mm_M3
- removed Ref** (x4): Val**, kbd:HOLE
- added G***: LOGO, lib:panda-throughhole, B.Cu at (67.0, 87.2)
- added H1: MountingHole, MountingHole:MountingHole_3.2mm_M3, F.Cu at (42.9, 45.2)
- added H2: MountingHole, MountingHole:MountingHole_3.2mm_M3, F.Cu at (100.0, 45.2)
- added H3: MountingHole, MountingHole:MountingHole_3.2mm_M3, F.Cu at (42.9, 102.4)
- added H4: MountingHole, MountingHole:MountingHole_3.2mm_M3, F.Cu at (100.0, 102.4)
- added H5: MountingHole, kbd:HOLE, F.Cu at (42.9, 64.3)
- added H6: MountingHole, kbd:HOLE, F.Cu at (100.0, 64.3)
- added H7: MountingHole, kbd:HOLE, F.Cu at (38.1, 102.4)
- added H8: MountingHole, kbd:HOLE, F.Cu at (104.8, 102.4)
- U1, U2: footprint Package_SO:SOIC-28W_7.5x17.9mm_P1.27mm -> Package_DIP:DIP-28_W7.62mm_Socket
- moved U1 24.1 mm to (35.7, 40.5)
- moved SW22 14.8 mm to (87.3, 27.5), turned to 180 degrees
- moved R1 14.1 mm to (53.0, 27.5), turned to 0 degrees
- moved SW21 11.7 mm to (97.5, 27.5), turned to 180 degrees
- moved U2 9.66 mm to (73.8, 40.5)
- moved D1 9.09 mm to (46.7, 27.5)
- moved J1 6.74 mm to (28.6, 26.2)
- moved C1 5.98 mm to (69.5, 27.5), turned to 0 degrees
- moved J2 5.32 mm to (114.3, 26.2)
Connections:
- U1 pad 1: SW6 -> SW11
- U1 pad 2: SW7 -> SW12
- U1 pad 21: SW5 -> SW3
- U1 pad 23: SW3 -> SW5
- U1 pad 3: SW8 -> SW13
- U1 pad 4: SW9 -> SW14
- U1 pad 5: SW10 -> SW15
- U2 pad 21: SW15 -> SW10
- U2 pad 22: SW14 -> SW9
- U2 pad 23: SW13 -> SW8
- U2 pad 24: SW12 -> SW7
- U2 pad 25: SW11 -> SW6
Routing:
- net GND: track 131.8 -> 32.0 mm, vias 6 -> 0
- net 3V3: track 108.2 -> 164.5 mm, vias 5 -> 1
- net SW7: track 42.8 -> 98.9 mm, vias 1 -> 2
- net SW6: track 45.8 -> 87.1 mm, vias 1 -> 2
- net SW20: track 122.4 -> 90.9 mm
- net SW19: track 104.4 -> 76.5 mm
- net SW5: track 61.5 -> 88.9 mm, vias 1 -> 0
- net SW11: track 93.6 -> 66.7 mm
- net SW8: track 54.3 -> 79.8 mm, vias 1 -> 2
- net SW4: track 46.9 -> 67.4 mm, vias 1 -> 0
- net SW15: track 91.0 -> 102.7 mm
- net SW13: track 80.2 -> 71.8 mm
- net SW17: track 112.7 -> 105.0 mm
- net SW18: track 114.3 -> 107.1 mm
- net SW1: track 39.0 -> 31.9 mm, vias 1 -> 0
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Other:
- board size 95.2 x 92.9 mm -> 95.2 x 97.6 mm
- board text added: "A1"
- board text added: "A2"
- board text added: "GND"
- board text added: "VCC"
