File: next-keyboard.sch (KiCad schematic (older format))
At the start: 29 parts, among them J1 MJ-4PP-9, J2 MJ-4PP-9, SW1 SW_PUSH, SW10 SW_PUSH, SW11 SW_PUSH, SW12 SW_PUSH, SW13 SW_PUSH, SW14 SW_PUSH, SW15 SW_PUSH, SW16 SW_PUSH, SW17 SW_PUSH, SW18 SW_PUSH, SW19 SW_PUSH, SW2 SW_PUSH, SW20 SW_PUSH, SW21 SW_SPDT, SW22 SW_SPDT, SW3 SW_PUSH, SW4 SW_PUSH, SW5 SW_PUSH, SW6 SW_PUSH, SW7 SW_PUSH, SW8 SW_PUSH, SW9 SW_PUSH, U1 MCP23017_SP, U2 MCP23017_SP

Commit message: produce
Parts:
- added H1, H2, H3, H4: MountingHole, MountingHole:MountingHole_3.2mm_M3, symbol Mechanical:MountingHole
- added H5, H6, H7, H8: MountingHole, kbd:HOLE, symbol Mechanical:MountingHole
- U1, U2: footprint Package_SO:SOIC-28W_7.5x17.9mm_P1.27mm -> Package_DIP:DIP-28_W7.62mm_Socket
Connections:
- net SW10: now also U2.21 (GPA0); no longer U1.5 (GPB4)
- net SW11: now also U1.1 (GPB0); no longer U2.25 (GPA4)
- net SW12: now also U1.2 (GPB1); no longer U2.24 (GPA3)
- net SW13: now also U1.3 (GPB2); no longer U2.23 (GPA2)
- net SW14: now also U1.4 (GPB3); no longer U2.22 (GPA1)
- net SW15: now also U1.5 (GPB4); no longer U2.21 (GPA0)
- net SW3: now also U1.21 (GPA0); no longer U1.23 (GPA2)
- net SW5: now also U1.23 (GPA2); no longer U1.21 (GPA0)
- net SW6: now also U2.25 (GPA4); no longer U1.1 (GPB0)
- net SW7: now also U2.24 (GPA3); no longer U1.2 (GPB1)
- net SW8: now also U2.23 (GPA2); no longer U1.3 (GPB2)
- net SW9: now also U2.22 (GPA1); no longer U1.4 (GPB3)
Changed lines of the file:
@@
 EESchema Schematic File Version 4
 LIBS:next-keyboard-cache
-EELAYER 26 0
+EELAYER 29 0
 EELAYER END
 $Descr A4 11693 8268
@@
 F 0 "U1" H 1950 3253 50  0000 C CNN
 F 1 "MCP23017_SP" H 1950 3162 50  0000 C CNN
-F 2 "Package_SO:SOIC-28W_7.5x17.9mm_P1.27mm" H 2150 975 50  0001 L CNN
+F 2 "Package_DIP:DIP-28_W7.62mm_Socket" H 2150 975 50  0001 L CNN
 F 3 "http://ww1.microchip.com/downloads/en/DeviceDoc/20001952C.pdf" H 2150 875 50  0001 L CNN
 	1    1950 1975
@@
 	1    0    0    -1
 $EndComp
-Text GLabel 1850 1275 1    50   Input ~ 0
+Text GLabel 1650 1275 1    50   Input ~ 0
 SW5
 Text GLabel 1750 1275 1    50   Input ~ 0
 SW4
-Text GLabel 1650 1275 1    50   Input ~ 0
+Text GLabel 1850 1275 1    50   Input ~ 0
 SW3
 Text GLabel 1550 1275 1    50   Input ~ 0
@@
 Text GLabel 1450 1275 1    50   Input ~ 0
 SW1
-Text GLabel 1150 2675 3    50   Input ~ 0
+Text GLabel 4075 1275 1    50   Input ~ 0
 SW6
-Text GLabel 1250 2675 3    50   Input ~ 0
+Text GLabel 4175 1275 1    50   Input ~ 0
 SW7
-Text GLabel 1350 2675 3    50   Input ~ 0
+Text GLabel 4275 1275 1    50   Input ~ 0
 SW8
-Text GLabel 1450 2675 3    50   Input ~ 0
+Text GLabel 4375 1275 1    50   Input ~ 0
 SW9
-Text GLabel 1550 2675 3    50   Input ~ 0
+Text GLabel 4475 1275 1    50   Input ~ 0
 SW10
 NoConn ~ 2100 1275
@@
 F 0 "U2" H 4575 3253 50  0000 C CNN
 F 1 "MCP23017_SP" H 4575 3162 50  0000 C CNN
-F 2 "Package_SO:SOIC-28W_7.5x17.9mm_P1.27mm" H 4775 975 50  0001 L CNN
+F 2 "Package_DIP:DIP-28_W7.62mm_Socket" H 4775 975 50  0001 L CNN
 F 3 "http://ww1.microchip.com/downloads/en/DeviceDoc/20001952C.pdf" H 4775 875 50  0001 L CNN
 	1    4575 1975
@@
 	1    0    0    -1
 $EndComp
-Text GLabel 4475 1275 1    50   Input ~ 0
+Text GLabel 1550 2675 3    50   Input ~ 0
 SW15
-Text GLabel 4375 1275 1    50   Input ~ 0
+Text GLabel 1450 2675 3    50   Input ~ 0
 SW14
-Text GLabel 4275 1275 1    50   Input ~ 0
+Text GLabel 1350 2675 3    50   Input ~ 0
 SW13
-Text GLabel 4175 1275 1    50   Input ~ 0
+Text GLabel 1250 2675 3    50   Input ~ 0
 SW12
-Text GLabel 4075 1275 1    50   Input ~ 0
+Text GLabel 1150 2675 3    50   Input ~ 0
 SW11
 Text GLabel 3775 2675 3    50   Input ~ 0
@@
 	0    1    1    0
 $EndComp
+$Comp
+L Mechanical:MountingHole H1
+U 1 1 5C63E87E
+P 6800 5200
+F 0 "H1" H 6900 5246 50  0000 L CNN
+F 1 "MountingHole" H 6900 5155 50  0000 L CNN
+F 2 "MountingHole:MountingHole_3.2mm_M3" H 6800 5200 50  0001 C CNN
+F 3 "~" H 6800 5200 50  0001 C CNN
+	1    6800 5200
+	1    0    0    -1
+$EndComp
+$Comp
+L Mechanical:MountingHole H2
+U 1 1 5C63E9D0
+P 7475 5200
+F 0 "H2" H 7575 5246 50  0000 L CNN
+F 1 "MountingHole" H 7575 5155 50  0000 L CNN
+F 2 "MountingHole:MountingHole_3.2mm_M3" H 7475 5200 50  0001 C CNN
+F 3 "~" H 7475 5200 50  0001 C CNN
+	1    7475 5200
+	1    0    0    -1
+$EndComp
+$Comp
+L Mechanical:MountingHole H4
+U 1 1 5C63EA73
+P 6800 5525
+F 0 "H4" H 6900 5571 50  0000 L CNN
+F 1 "MountingHole" H 6900 5480 50  0000 L CNN
+F 2 "MountingHole:MountingHole_3.2mm_M3" H 6800 5525 50  0001 C CNN
+F 3 "~" H 6800 5525 50  0001 C CNN
+	1    6800 5525
+	1    0    0    -1
+$EndComp
+$Comp
+L Mechanical:MountingHole H3
+U 1 1 5C63EB03
+P 7500 5500
+F 0 "H3" H 7600 5546 50  0000 L CNN
+F 1 "MountingHole" H 7600 5455 50  0000 L CNN
+F 2 "MountingHole:MountingHole_3.2mm_M3" H 7500 5500 50  0001 C CNN
+F 3 "~" H 7500 5500 50  0001 C CNN
+	1    7500 5500
+	1    0    0    -1
+$EndComp
+$Comp
+L Mechanical:MountingHole H6
+U 1 1 5C63EB90
+P 6800 5825
+F 0 "H6" H 6900 5871 50  0000 L CNN
+F 1 "MountingHole" H 6900 5780 50  0000 L CNN
+F 2 "kbd:HOLE" H 6800 5825 50  0001 C CNN
+F 3 "~" H 6800 5825 50  0001 C CNN
+	1    6800 5825
+	1    0    0    -1
+$EndComp
+$Comp
+L Mechanical:MountingHole H5
+U 1 1 5C63EC1E
+P 7525 5800
+F 0 "H5" H 7625 5846 50  0000 L CNN
+F 1 "MountingHole" H 7625 5755 50  0000 L CNN
+F 2 "kbd:HOLE" H 7525 5800 50  0001 C CNN
+F 3 "~" H 7525 5800 50  0001 C CNN
+	1    7525 5800
+	1    0    0    -1
+$EndComp
+$Comp
+L Mechanical:MountingHole H7
+U 1 1 5C63ECAF
+P 6800 6075
+F 0 "H7" H 6900 6121 50  0000 L CNN
+F 1 "MountingHole" H 6900 6030 50  0000 L CNN
+F 2 "kbd:HOLE" H 6800 6075 50  0001 C CNN
+F 3 "~" H 6800 6075 50  0001 C CNN
+	1    6800 6075
+	1    0    0    -1
+$EndComp
+$Comp
+L Mechanical:MountingHole H8
+U 1 1 5C63ED73
+P 7525 6075
+F 0 "H8" H 7625 6121 50  0000 L CNN
+F 1 "MountingHole" H 7625 6030 50  0000 L CNN
+F 2 "kbd:HOLE" H 7525 6075 50  0001 C CNN
+F 3 "~" H 7525 6075 50  0001 C CNN
+	1    7525 6075
+	1    0    0    -1
+$EndComp
 $EndSCHEMATC
